Commit message: Added basic igvc, c920, and hokuyo descriptions

File: ucf_igvc/src/igvc/igvc_description/tests/wheel_only_test.urdf.xacro (robot description, xacro)
@@ -3,4 +3,7 @@
 	<!-- Include full igvc library even though we're not using all of it -->
 	<xacro:include filename="$(find igvc_description)/urdf/igvc_library.urdf.xacro"/>
+	<xacro:include filename="$(find igvc_description)/urdf/igvc_materials.urdf.xacro"/>
+	<xacro:include filename="$(find core_description)/urdf/sensors/cameras/c920_camera.urdf.xacro"/>
+	<xacro:include filename="$(find core_description)/urdf/sensors/lasers/hokuyo.urdf.xacro"/>
 	<!-- Base link -->
 	<link name="base_link">
@@ -20,9 +23,42 @@
 			<inertia ixx="0.05" ixy="0" ixz="0" iyy="0.05" iyz="0" izz="0.05"/>
 		</inertial>
+		<!-- Gazebo description for base_link -->
+		<gazebo reference="base_link"/>
 	</link>
-	<!-- Gazebo description for base_link -->
-	<gazebo reference="base_link"/>
+	<!-- Base footprint as a reference to the ground beneath robot -->
+	<link name="base_footprint">
+		<visual>
+			<geometry>
+				<box size="0.001 0.001 0.001"/>
+			</geometry>
+			<origin xyz="0 0 0" rpy="0 0 0"/>
+		</visual>
+		<inertial>
+			<mass value="0.0001"/>
+			<origin xyz="0 0 0"/>
+			<inertia ixx="0.0001" ixy="0.0" ixz="0.0" iyy="0.0001" iyz="0.0" izz="0.0001"/>
+		</inertial>
+		<gazebo reference="base_footprint"/>
+	</link>
+	<!-- Joint connecting base_link to the footprint -->
+	<joint name="base_footprint_joint" type="fixed">
+		<origin xyz="0 0 0.06"/>
+		<parent link="base_footprint"/>
+		<child link="base_link"/>
+		<gazebo reference="base_footprint_joint"/>
+	</joint>
 	<!-- Add the wheels -->
 	<igvc_wheel parent="base_link" lr="right" reflectY="-1"/>
 	<igvc_wheel parent="base_link" lr="left" reflectY="1"/>
+	<!-- Add the casters -->
+	<igvc_caster parent="base_link" lr="right" reflectY="-1"/>
+	<igvc_caster parent="base_link" lr="left" reflectY="1"/>
+	<!-- Add a camera -->
+	<c920_camera identifier="solo" parent="base_link" xPos="0.1" yPos="0.0" zPos="0.1" roll="0" pitch="0.4" yaw="0"/>
+	<c920_camera identifier="double" parent="base_link" xPos="-0.1" yPos="0.0" zPos="0.1" roll="0" pitch="0.4" yaw="3.14159"/>
+	<!-- Add a laser -->
+	<hokuyo_utm30lx parent="base_link" xPos="0.1" yPos="0.1" zPos="0.1" roll="0" pitch="0" yaw="0"/>
+	<!-- Set up miscellaneous igvc plugins not related to sensors -->
+	<igvc_gazebo />
+	<gazebo reference="igvc"/>
 </robot>

File: ucf_igvc/src/igvc/igvc_description/urdf/igvc_library.urdf.xacro (robot description, xacro)
@@ -5,3 +5,7 @@
 	<!-- IGVC wheel description -->
 	<xacro:include filename="$(find igvc_description)/urdf/igvc_wheel.urdf.xacro"/>
+	<!-- IGVC caster description -->
+	<xacro:include filename="$(find igvc_description)/urdf/igvc_caster.urdf.xacro"/>
+	<!-- IGVC gazebo description -->
+	<xacro:include filename="$(find igvc_description)/urdf/igvc_gazebo.urdf.xacro"/>
 </robot>

File: ucf_igvc/src/igvc/igvc_description/urdf/igvc_properties.urdf.xacro (robot description, xacro)
@@ -7,13 +7,28 @@
 	<property name="wheel_mass" value="5"/>
 	<property name="wheel_width" value="0.02"/>
-	<property name="wheel_radius" value="0.02"/>
+	<property name="wheel_radius" value="0.06"/>
 	<property name="wheel_ixx" value="${(wheel_mass*(3*wheel_radius*wheel_radius + wheel_width*wheel_width))/12}"/>
 	<property name="wheel_iyy" value="${(wheel_mass*(3*wheel_radius*wheel_radius + wheel_width*wheel_width))/12}"/>
 	<property name="wheel_izz" value="${(wheel_mass*wheel_radius*wheel_radius)/2}"/>
 	<property name="wheel_x_pos" value="0"/>
-	<property name="wheel_y_pos" value="0.1"/>
+	<property name="wheel_y_pos" value="${0.1 + wheel_width/2}"/>
 	<property name="wheel_z_pos" value="-0.1"/>
 	<!-- Caster properties -->
-	<!-- Camera properties -->
+	<property name="caster_wheel_mass" value="5"/>
+	<property name="caster_wheel_width" value="0.02"/>
+	<property name="caster_wheel_radius" value="0.02"/>
+	<property name="caster_wheel_ixx" value="${(caster_wheel_mass*(3*caster_wheel_radius*caster_wheel_radius + caster_wheel_width*caster_wheel_width))/12}"/>
+	<property name="caster_wheel_iyy" value="${(caster_wheel_mass*(3*caster_wheel_radius*caster_wheel_radius + caster_wheel_width*caster_wheel_width))/12}"/>
+	<property name="caster_wheel_izz" value="${(caster_wheel_mass*caster_wheel_radius*caster_wheel_radius)/2}"/>
+	<!-- Caster rotator properties -->
+	<property name="caster_rotator_mass" value="1"/>
+	<property name="caster_rotator_width" value="0.001"/>
+	<property name="caster_rotator_radius" value="${caster_wheel_radius}"/>
+	<property name="caster_rotator_ixx" value="0.001"/>
+	<property name="caster_rotator_iyy" value="0.001"/>
+	<property name="caster_rotator_izz" value="0.001"/>
+	<property name="caster_x_pos" value="0.08"/>
+	<property name="caster_y_pos" value="0.02"/>
+	<property name="caster_z_pos" value="-0.1"/>
 	<!-- LIDAR properties -->
 </robot>

File: ucf_igvc/src/igvc/igvc_description/urdf/igvc_wheel.urdf.xacro (robot description, xacro)
@@ -3,5 +3,4 @@
 	<!-- Include IGVC vehicle properties -->
 	<xacro:include filename="$(find igvc_description)/urdf/igvc_properties.urdf.xacro"/>
-	<xacro:include filename="$(find igvc_description)/urdf/igvc_materials.urdf.xacro"/>
 	<!-- Macro providing complete description of a wheel, joint, and motor -->
 	<!-- A differential drive is assumed here. -->
@@ -12,4 +11,5 @@
 			<visual>
 				<geometry>
+					<!-- Change to mesh when we have them??? -->
 					<cylinder length="${wheel_width}" radius="${wheel_radius}"/>
 				</geometry>

Commit message: added super broken nav stack stuff

File: ucf_igvc/src/igvc/igvc_description/tests/wheel_only_test.urdf.xacro (robot description, xacro)
@@ -6,20 +6,20 @@
 	<xacro:include filename="$(find core_description)/urdf/sensors/cameras/c920_camera.urdf.xacro"/>
 	<xacro:include filename="$(find core_description)/urdf/sensors/lasers/hokuyo.urdf.xacro"/>
+	<xacro:include filename="$(find igvc_description)/urdf/igvc_properties.urdf.xacro"/>
 	<!-- Base link -->
 	<link name="base_link">
 		<visual>
 			<geometry>
-				<box size="0.2 0.2 0.2"/>
+				<box size="${chassis_length} ${chassis_width} ${chassis_height}"/>
 			</geometry>
-			<material name="white"/>
 		</visual>
 		<collision>
 			<geometry>
-				<box size="0.1 0.2 0.2"/>
+				<box size="${chassis_length} ${chassis_width} ${chassis_height}"/>
 			</geometry>
 		</collision>
 		<inertial>
-			<mass value="10"/>
-			<inertia ixx="0.05" ixy="0" ixz="0" iyy="0.05" iyz="0" izz="0.05"/>
+			<mass value="${chassis_mass}"/>
+			<inertia ixx="${chassis_ixx}" ixy="0" ixz="0" iyy="${chassis_iyy}" iyz="0" izz="${chassis_izz}"/>
 		</inertial>
 		<!-- Gazebo description for base_link -->
@@ -43,5 +43,5 @@
 	<!-- Joint connecting base_link to the footprint -->
 	<joint name="base_footprint_joint" type="fixed">
-		<origin xyz="0 0 0.06"/>
+		<origin xyz="0 0 ${chassis_height/2}"/>
 		<parent link="base_footprint"/>
 		<child link="base_link"/>
@@ -55,8 +55,8 @@
 	<igvc_caster parent="base_link" lr="left" reflectY="1"/>
 	<!-- Add a camera -->
-	<c920_camera identifier="solo" parent="base_link" xPos="0.1" yPos="0.0" zPos="0.1" roll="0" pitch="0.4" yaw="0"/>
-	<c920_camera identifier="double" parent="base_link" xPos="-0.1" yPos="0.0" zPos="0.1" roll="0" pitch="0.4" yaw="3.14159"/>
+	<c920_camera identifier="solo" parent="base_link" xPos="${chassis_length/2}" yPos="0" zPos="${chassis_height/2}" roll="0" pitch="0.4" yaw="0"/>
+	<c920_camera identifier="double" parent="base_link" xPos="-${chassis_length/2}" yPos="0.0" zPos="${chassis_height/2}" roll="0" pitch="0.4" yaw="3.14159"/>
 	<!-- Add a laser -->
-	<hokuyo_utm30lx parent="base_link" xPos="0.1" yPos="0.1" zPos="0.1" roll="0" pitch="0" yaw="0"/>
+	<hokuyo_utm30lx parent="base_link" xPos="0" yPos="0" zPos="${chassis_height/2 + 0.2}" roll="0" pitch="-0.01" yaw="0"/>
 	<!-- Set up miscellaneous igvc plugins not related to sensors -->
 	<igvc_gazebo />

File: ucf_igvc/src/igvc/igvc_description/urdf/igvc_gazebo.urdf.xacro (robot description, xacro)
@@ -12,7 +12,7 @@
 				<leftJoint>left_wheel_joint</leftJoint>
 				<rightJoint>right_wheel_joint</rightJoint>
-				<wheelSeparation>${0.2 + wheel_width/2}</wheelSeparation>
+				<wheelSeparation>${chassis_width + wheel_width/2}</wheelSeparation>
 				<wheelDiameter>${2*wheel_radius}</wheelDiameter>
-				<wheelTorque>10</wheelTorque>
+				<wheelTorque>27</wheelTorque>
 				<robotBaseFrame>base_footprint</robotBaseFrame>
 				<odometryFrame>map</odometryFrame>

File: ucf_igvc/src/igvc/igvc_description/urdf/igvc_properties.urdf.xacro (robot description, xacro)
@@ -4,18 +4,25 @@
 	<property name="M_PI" value="3.14159"/>
 	<!-- Chassis properties -->
+	<property name="chassis_mass" value="62"/>
+	<property name="chassis_length" value="1.14"/>
+	<property name="chassis_width" value="0.559"/>
+	<property name="chassis_height" value="0.5"/>
+	<property name="chassis_ixx" value="${(chassis_mass*(chassis_length*chassis_length+chassis_height*chassis_height))/12}"/>
+	<property name="chassis_iyy" value="${(chassis_mass*(chassis_height*chassis_height+chassis_width*chassis_width))/12}"/>
+	<property name="chassis_izz" value="${(chassis_mass*(chassis_width*chassis_width+chassis_length*chassis_length))/12}"/>
 	<!-- Wheel properties -->
-	<property name="wheel_mass" value="5"/>
-	<property name="wheel_width" value="0.02"/>
-	<property name="wheel_radius" value="0.06"/>
+	<property name="wheel_mass" value="3.4"/>
+	<property name="wheel_width" value="0.127"/>
+	<property name="wheel_radius" value="0.153"/>
 	<property name="wheel_ixx" value="${(wheel_mass*(3*wheel_radius*wheel_radius + wheel_width*wheel_width))/12}"/>
 	<property name="wheel_iyy" value="${(wheel_mass*(3*wheel_radius*wheel_radius + wheel_width*wheel_width))/12}"/>
 	<property name="wheel_izz" value="${(wheel_mass*wheel_radius*wheel_radius)/2}"/>
-	<property name="wheel_x_pos" value="0"/>
-	<property name="wheel_y_pos" value="${0.1 + wheel_width/2}"/>
-	<property name="wheel_z_pos" value="-0.1"/>
+	<property name="wheel_x_pos" value="-${chassis_length/2 - wheel_radius - 0.05}"/>
+	<property name="wheel_y_pos" value="${0.3 + wheel_width/2}"/>
+	<property name="wheel_z_pos" value="-${chassis_height/2 + 0.1}"/>
 	<!-- Caster properties -->
-	<property name="caster_wheel_mass" value="5"/>
-	<property name="caster_wheel_width" value="0.02"/>
-	<property name="caster_wheel_radius" value="0.02"/>
+	<property name="caster_wheel_mass" value="2"/>
+	<property name="caster_wheel_width" value="0.071"/>
+	<property name="caster_wheel_radius" value="0.101"/>
 	<property name="caster_wheel_ixx" value="${(caster_wheel_mass*(3*caster_wheel_radius*caster_wheel_radius + caster_wheel_width*caster_wheel_width))/12}"/>
 	<property name="caster_wheel_iyy" value="${(caster_wheel_mass*(3*caster_wheel_radius*caster_wheel_radius + caster_wheel_width*caster_wheel_width))/12}"/>
@@ -28,7 +35,7 @@
 	<property name="caster_rotator_iyy" value="0.001"/>
 	<property name="caster_rotator_izz" value="0.001"/>
-	<property name="caster_x_pos" value="0.08"/>
-	<property name="caster_y_pos" value="0.02"/>
-	<property name="caster_z_pos" value="-0.1"/>
+	<property name="caster_x_pos" value="${chassis_length/2 - 2*caster_wheel_radius}"/>
+	<property name="caster_y_pos" value="${chassis_width/4}"/>
+	<property name="caster_z_pos" value="-${chassis_height/2 + 0.025}"/>
 	<!-- LIDAR properties -->
 </robot>

Commit message: starting over on navstack params

File: ucf_igvc/src/igvc/igvc_description/tests/wheel_only_test.urdf.xacro (robot description, xacro)
@@ -11,5 +11,5 @@
 		<visual>
 			<geometry>
-				<box size="${chassis_length} ${chassis_width} ${chassis_height}"/>
+				<mesh filename="package://igvc_description/meshes/igvc_chassis.DAE" scale="0.85 0.75 0.90"/>
 			</geometry>
 		</visual>

File: ucf_igvc/src/igvc/igvc_description/urdf/igvc_properties.urdf.xacro (robot description, xacro)
@@ -7,5 +7,5 @@
 	<property name="chassis_length" value="1.14"/>
 	<property name="chassis_width" value="0.559"/>
-	<property name="chassis_height" value="0.5"/>
+	<property name="chassis_height" value="0.42"/>
 	<property name="chassis_ixx" value="${(chassis_mass*(chassis_length*chassis_length+chassis_height*chassis_height))/12}"/>
 	<property name="chassis_iyy" value="${(chassis_mass*(chassis_height*chassis_height+chassis_width*chassis_width))/12}"/>
