Commit message: polishing up description and navstack files

File: ucf_core/src/core/core_description/urdf/sensors/lasers/hokuyo.urdf.xacro (robot description, xacro)
@@ -31,13 +31,13 @@
             <sensor type="ray" name="laser">
                 <pose>0 0 0 0 0 0</pose>
-                <visualize>false</visualize>
+                <visualize>true</visualize>
                 <update_rate>40</update_rate>
                 <ray>
                     <scan>
                         <horizontal>
-                            <samples>720</samples>
+                            <samples>1080</samples>
                             <resolution>1</resolution>
-                            <min_angle>-1.570796</min_angle>
-                            <max_angle>1.570796</max_angle>
+                            <min_angle>-2.3562</min_angle>
+                            <max_angle>2.3562</max_angle>
                         </horizontal>
                     </scan>
@@ -48,5 +48,5 @@
                     </range>
                     <noise>
-                        <type>Gaussian</type>
+                        <type>gaussian</type>
                         <mean>0.0</mean>
                         <stddev>0.01</stddev>

File: ucf_igvc/src/igvc/igvc_description/robots/igvc.urdf.xacro (robot description, xacro)
@@ -11,10 +11,10 @@
 		<visual>
 			<geometry>
-				<mesh filename="package://igvc_description/meshes/igvc_chassis.DAE" scale="1 0.90 1" />
+				<mesh filename="package://igvc_description/meshes/igvc_chassis.DAE" scale="1 1 1" />
 			</geometry>
 		</visual>
 		<collision>
 			<geometry>
-				<box size="${chassis_length} ${chassis_width} ${chassis_height}"/>
+				<mesh filename="package://igvc_description/meshes/igvc_chassis.DAE" scale="1 1 1" />
 			</geometry>
 		</collision>
@@ -55,9 +55,9 @@
 	<igvc_caster parent="base_link" lr="left" reflectY="1"/>
 	<!-- Add a camera -->
-	<c920_camera identifier="one" parent="base_link" xPos="-0.6" yPos="0.05" zPos="1.2" roll="0" pitch="0.35" yaw="1.57057"/>
-	<c920_camera identifier="two" parent="base_link" xPos="-0.5" yPos="0.0" zPos="1.2" roll="0" pitch="0.35" yaw="0"/>
-	<c920_camera identifier="three" parent="base_link" xPos="-0.6" yPos="-0.05" zPos="1.2" roll="0" pitch="0.35" yaw="-1.57057"/>
+	<c920_camera identifier="left" parent="base_link" xPos="-0.6" yPos="0.05" zPos="1.2" roll="0" pitch="0.35" yaw="1.57057"/>
+	<c920_camera identifier="front" parent="base_link" xPos="-0.5" yPos="0.0" zPos="1.2" roll="0" pitch="0.35" yaw="0"/>
+	<c920_camera identifier="right" parent="base_link" xPos="-0.6" yPos="-0.05" zPos="1.2" roll="0" pitch="0.35" yaw="-1.57057"/>
 	<!-- Add a laser -->
-	<hokuyo_utm30lx parent="base_link" xPos="0.45" yPos="0" zPos="0" roll="0" pitch="-0.01" yaw="0"/>
+	<hokuyo_utm30lx parent="base_link" xPos="0.62" yPos="0" zPos="-0.26" roll="0" pitch="0" yaw="0"/>
 	<!-- Set up miscellaneous igvc plugins not related to sensors -->
 	<igvc_gazebo />

File: ucf_igvc/src/igvc/igvc_description/urdf/igvc_properties.urdf.xacro (robot description, xacro)
@@ -19,10 +19,10 @@
 	<property name="wheel_izz" value="${(wheel_mass*wheel_radius*wheel_radius)/2}"/>
 	<property name="wheel_x_pos" value="-${chassis_length/2 - wheel_radius - 0.05}"/>
-	<property name="wheel_y_pos" value="${0.3 + wheel_width/2}"/>
+	<property name="wheel_y_pos" value="${0.3048 + wheel_width/2}"/>
 	<property name="wheel_z_pos" value="-${chassis_height/2 + 0.1}"/>
 	<!-- Caster properties -->
 	<property name="caster_wheel_mass" value="2"/>
 	<property name="caster_wheel_width" value="0.071"/>
-	<property name="caster_wheel_radius" value="0.101"/>
+	<property name="caster_wheel_radius" value="0.107"/>
 	<property name="caster_wheel_ixx" value="${(caster_wheel_mass*(3*caster_wheel_radius*caster_wheel_radius + caster_wheel_width*caster_wheel_width))/12}"/>
 	<property name="caster_wheel_iyy" value="${(caster_wheel_mass*(3*caster_wheel_radius*caster_wheel_radius + caster_wheel_width*caster_wheel_width))/12}"/>
