Commit message: Vastly improved navigation stack functionality and added rviz convenience launchers

File: ucf_core/src/core/core_description/urdf/sensors/cameras/c920_camera.urdf.xacro (robot description, xacro)
@@ -22,5 +22,4 @@
 					<box size="${c920_length} ${c920_width} ${c920_height}"/>
 				</geometry>
-				<origin rpy="${roll} ${pitch} ${yaw}"/>
 			</collision>
 			<inertial>
@@ -35,5 +34,5 @@
 				<update_rate>30.0</update_rate>
 				<camera name="${identifier}">
-					<horizontal_fov>1.57057</horizontal_fov>
+					<horizontal_fov>1.05</horizontal_fov>
 					<image>
 						<width>1920</width>

File: ucf_core/src/core/core_description/urdf/sensors/lasers/hokuyo.urdf.xacro (robot description, xacro)
@@ -31,5 +31,5 @@
             <sensor type="ray" name="laser">
                 <pose>0 0 0 0 0 0</pose>
-                <visualize>true</visualize>
+                <visualize>false</visualize>
                 <update_rate>40</update_rate>
                 <ray>
@@ -47,9 +47,4 @@
                         <resolution>0.01</resolution>
                     </range>
-                    <noise>
-                        <type>gaussian</type>
-                        <mean>0.0</mean>
-                        <stddev>0.01</stddev>
-                    </noise>
                 </ray>
                 <plugin name="hokuyo_node" filename="libgazebo_ros_laser.so">
