Commit message: Add basic non-simulation robot launch.
* Adds launch file for non-simulation robot.
* Rearranges some existing configuration files.
* Change frame in csi_minimax launch to gps from minimax_gps.

File: ucf_core/src/core/core_description/urdf/sensors/gps/csi_minimax.urdf.xacro (robot description, xacro)
@@ -6,5 +6,5 @@
     <xacro:property name="minimax_height" value="0.025" />
     <xacro:macro name="minimax_gps" params="parent xPos yPos zPos roll pitch yaw" >
-        <link name="minimax_gps" >
+        <link name="gps" >
             <visual>
                 <origin xyz="0 0 0" rpy="0 0 0" />
@@ -27,11 +27,11 @@
             </inertial>
         </link>
-        <gazebo reference="minimax_gps" />
-        <joint name="minimax_gps_joint" type="fixed" >
+        <gazebo reference="gps" />
+        <joint name="gps_joint" type="fixed" >
             <parent link="${parent}" />
-            <child link="minimax_gps" />
+            <child link="gps" />
             <origin xyz="${xPos} ${yPos} ${zPos}" rpy="${roll} ${pitch} ${yaw}" />
         </joint>
-        <gazebo reference="minimax_gps_joint" />
+        <gazebo reference="gps_joint" />
     </xacro:macro>
 </robot>

File: ucf_igvc/src/igvc/igvc_description/robots/igvc.urdf.xacro (robot description, xacro)
@@ -57,11 +57,11 @@
 	<igvc_caster parent="base_link" lr="left" reflectY="1"/>
 	<!-- Add a camera -->
-	<c920_camera identifier="left" parent="base_link" xPos="-0.6" yPos="0.05" zPos="1.2" roll="0" pitch="0.35" yaw="1.57057"/>
+	<c920_camera identifier="left" parent="base_link" xPos="-0.6" yPos="0.05" zPos="1.2" roll="0" pitch="0.35" yaw="1.5708"/>
 	<c920_camera identifier="front" parent="base_link" xPos="-0.5" yPos="0.0" zPos="1.2" roll="0" pitch="0.35" yaw="0"/>
-	<c920_camera identifier="right" parent="base_link" xPos="-0.6" yPos="-0.05" zPos="1.2" roll="0" pitch="0.35" yaw="-1.57057"/>
+	<c920_camera identifier="right" parent="base_link" xPos="-0.6" yPos="-0.05" zPos="1.2" roll="0" pitch="0.35" yaw="-1.5708"/>
 	<!-- Add a laser -->
-	<hokuyo_utm30lx parent="base_link" xPos="0.62" yPos="0" zPos="-0.26" roll="0" pitch="0" yaw="0"/>
+	<hokuyo_utm30lx parent="base_link" xPos="0.62" yPos="0" zPos="-0.26" roll="3.14159" pitch="0" yaw="0"/>
 	<!-- Add AHRS-8 -->
-	<sparton_ahrs8 parent="base_link" xPos="0.0" yPos="0" zPos="0.2" roll="0" pitch="0" yaw="0"/>
+	<sparton_ahrs8 parent="base_link" xPos="0.0" yPos="0" zPos="0.2" roll="0" pitch="-1.5708" yaw="3.14159"/>
 	<!-- Add GPS -->
 	<minimax_gps parent="base_link" xPos="-0.2" yPos="0" zPos="0.2" roll="0" pitch="0" yaw="0" />
