Commit message: Updating some confliguration files to incorporate vision and laser merging.

File: ucf_igvc/src/igvc/igvc_description/robots/igvc.urdf.xacro (robot description, xacro)
@@ -50,4 +50,18 @@
 		<gazebo reference="base_footprint_joint"/>
 	</joint>
+	<!-- Attach front_front_fake_laser frame -->
+	<link name="front_fake_laser">
+		<visual>
+			<geometry>
+				<box size="0.001 0.001 0.001" />
+			</geometry>
+			<origin xyz="0 0 0" rpy="0 0 0"/>
+		</visual>
+	</link>
+	<joint name="front_fake_laser_joint" type="fixed">
+		<origin xyz="0.8 0 0"/>
+		<parent link="base_link"/>
+		<child link="front_fake_laser"/>
+	</joint>
 	<!-- Add the wheels -->
 	<igvc_wheel parent="base_link" lr="right" reflectY="-1"/>
@@ -61,5 +75,5 @@
 	<c920_camera identifier="right" parent="base_link" xPos="-0.6" yPos="-0.05" zPos="1.2" roll="0" pitch="0.35" yaw="-1.5708"/>
 	<!-- Add a laser -->
-	<hokuyo_utm30lx parent="base_link" xPos="0.62" yPos="0" zPos="0" roll="3.14159" pitch="0" yaw="0"/>
+	<hokuyo_utm30lx parent="base_link" xPos="0.62" yPos="0" zPos="0" roll="0" pitch="0" yaw="0"/>
 	<!-- Add AHRS-8 -->
 	<sparton_ahrs8 parent="base_link" xPos="0.0" yPos="0" zPos="0" roll="0" pitch="0" yaw="0"/>

Commit message: Local changes to get approximate correct operation indoors -Kenneth

File: ucf_igvc/src/igvc/igvc_description/robots/igvc.urdf.xacro (robot description, xacro)
@@ -64,4 +64,30 @@
 		<child link="front_fake_laser"/>
 	</joint>
+	<link name="left_fake_laser">
+		<visual>
+			<geometry>
+				<box size="0.001 0.001 0.001" />
+			</geometry>
+			<origin xyz="0 0 0" rpy="0 0 0"/>
+		</visual>
+	</link>
+	<joint name="left_fake_laser_joint" type="fixed">
+		<origin xyz="0.33 0.737 0" rpy="0 0 0.7854"/>
+		<parent link="base_link"/>
+		<child link="left_fake_laser"/>
+	</joint>
+	<link name="right_fake_laser">
+		<visual>
+			<geometry>
+				<box size="0.001 0.001 0.001" />
+			</geometry>
+			<origin xyz="0 0 0" rpy="0 0 0"/>
+		</visual>
+	</link>
+	<joint name="right_fake_laser_joint" type="fixed">
+		<origin xyz="0.33 -0.737 0" rpy="0 0 -0.7854"/>
+		<parent link="base_link"/>
+		<child link="right_fake_laser"/>
+	</joint>
 	<!-- Add the wheels -->
 	<igvc_wheel parent="base_link" lr="right" reflectY="-1"/>

Commit message: Adjusting fake laser frames and limiting vsion to 15 fps -Kenneth

File: ucf_igvc/src/igvc/igvc_description/robots/igvc.urdf.xacro (robot description, xacro)
@@ -60,5 +60,5 @@
 	</link>
 	<joint name="front_fake_laser_joint" type="fixed">
-		<origin xyz="0.8 0 0"/>
+		<origin xyz="0.95 0 0"/>
 		<parent link="base_link"/>
 		<child link="front_fake_laser"/>

Commit message: Pushing field changes

File: ucf_igvc/src/igvc/igvc_description/robots/igvc.urdf.xacro (robot description, xacro)
@@ -60,5 +60,5 @@
 	</link>
 	<joint name="front_fake_laser_joint" type="fixed">
-		<origin xyz="0.95 0 0"/>
+		<origin xyz="1.2 0 0"/>
 		<parent link="base_link"/>
 		<child link="front_fake_laser"/>
@@ -105,5 +105,5 @@
 	<sparton_ahrs8 parent="base_link" xPos="0.0" yPos="0" zPos="0" roll="0" pitch="0" yaw="0"/>
 	<!-- Add GPS -->
-	<minimax_gps parent="base_link" xPos="-0.2" yPos="0" zPos="0.2" roll="0" pitch="0" yaw="0" />
+	<minimax_gps parent="base_link" xPos="-0.4" yPos="0" zPos="0.8" roll="0" pitch="0" yaw="0" />
 	<!-- Set up miscellaneous igvc plugins not related to sensors -->
 	<igvc_gazebo />

Commit message: Pushing field changes -Kenneth

File: ucf_igvc/src/igvc/igvc_description/robots/igvc.urdf.xacro (robot description, xacro)
@@ -60,5 +60,5 @@
 	</link>
 	<joint name="front_fake_laser_joint" type="fixed">
-		<origin xyz="1.2 0 0"/>
+		<origin xyz="1.0 0 0"/>
 		<parent link="base_link"/>
 		<child link="front_fake_laser"/>
@@ -73,5 +73,5 @@
 	</link>
 	<joint name="left_fake_laser_joint" type="fixed">
-		<origin xyz="0.33 0.737 0" rpy="0 0 0.7854"/>
+		<origin xyz="0.49 0.845 0" rpy="0 0 0.7854"/>
 		<parent link="base_link"/>
 		<child link="left_fake_laser"/>
